File: SchaltplanETP2.sch (EAGLE design)
At the start: 66 parts, among them IC1 LM2674, IC2 ZXLD1350, IC3 ZXLD1350, IC4 ZXLD1350, IC5 ZXLD1350, M1 RN42_BLUETOOTH, T1 BUK98150-55A, X1 TERMINAL_BLOCK_MC000036, X2 TERMINAL_BLOCK_MC000036, X3 TERMINAL_BLOCK_MC000036

Commit message: added PCA9685 i2c to pwm 16 channel driver
Parts:
- removed JP8: (no value), adafruit:PINHD-1X8CLEANBIG
- added C20: 10uF, microbuilder:CAP_CERAMIC0805
- added R13, R14, R15, R16, R17, R18, R19, R20, R21: 10K, microbuilder:RESISTOR0805
- added SJ_A0, SJ_A1, SJ_A2, SJ_A3, SJ_A4, SJ_A5: (no value), microbuilder:SOLDERJUMPERREFLOW_NOPASTE
- added U1: PCA9685, microbuilder:PCA9685
Connections:
- removed net MCU_I2C: JP7.15, JP8.6
- removed net MCU_I2C2: JP7.16, JP8.7
- removed net N$28: JP8.8
- new net 4_PWM: U1.PWM4
- new net A0: R18.2, SJ_A0.2, U1.A0
- new net A1: R17.2, SJ_A1.2, U1.A1
- new net A2: R16.2, SJ_A2.2, U1.A2
- new net A3: R15.2, SJ_A3.2, U1.A3
- new net A4: R14.2, SJ_A4.2, U1.A4
- new net A5: R13.2, SJ_A5.2, U1.A5
- new net OE: R19.1, U1.#OE
- new net PWM10: U1.PWM10
- new net PWM11: U1.PWM11
- new net PWM12: U1.PWM12
- new net PWM13: U1.PWM13
- new net PWM14: U1.PWM14
- new net PWM15: U1.PWM15
- new net PWM6: U1.PWM6
- new net PWM7: U1.PWM7
- new net PWM8: U1.PWM8
- new net PWM9: U1.PWM9
- new net SCL: JP7.15, R21.1, U1.SCL
- new net SDA: JP7.16, R20.1, U1.SDA
- new net VCC: C20.P$1, R20.2, R21.2, SJ_A0.1, SJ_A1.1, SJ_A2.1, SJ_A3.1, SJ_A4.1, SJ_A5.1, U1.VDD
- net 0_PWM: now also U1.PWM0; no longer JP8.1
- net 1_PWM: now also U1.PWM1; no longer JP8.2
- net 2_PWM: now also U1.PWM2; no longer JP8.3
- net 3_PWM: now also U1.PWM3; no longer JP8.4
- net GND: now also C20.P$2, R13.1, R14.1, R15.1, R16.1, R17.1, R18.1, R19.2, U1.EXTCLK, U1.GND
- net M_PWM: now also U1.PWM5; no longer JP8.5
Other:
- note added: "1 + A5 + A4 + A3 + A2 + A1 +A1 + RW"
- note added: "Check sda scl polarity"
- note added: "I2C Address ="
- note added: "Open = 0 / Closed = 1"
- note removed: "MCU"

Commit message: rearrangement of the components
Parts:
- removed JP1: (no value), pinhead:PINHD-1X2
- removed R13, R14, R15, R16, R17, R18: 10K, microbuilder:RESISTOR0805
- removed SJ_A0, SJ_A1, SJ_A2, SJ_A3, SJ_A4, SJ_A5: (no value), microbuilder:SOLDERJUMPERREFLOW_NOPASTE
- removed X3: TERMINAL_BLOCK_MC000036, Moodlight:TERMINAL_BLOCK_MC000036
- added IR-RECEIVER: 22-23-2031, con-molex:22-23-2031
- added MOTOR: 22-23-2021, con-molex:22-23-2021
Connections:
- removed net +3V3: 0604.2, C3.2, C6.+, D1.A, IC1.FB, JP2.1, U$4.A
- removed net 4_PWM: U1.PWM4
- removed net 5V: JP5.1, JP6.1
- removed net A0: R18.2, SJ_A0.2, U1.A0
- removed net A1: R17.2, SJ_A1.2, U1.A1
- removed net A2: R16.2, SJ_A2.2, U1.A2
- removed net A3: R15.2, SJ_A3.2, U1.A3
- removed net A4: R14.2, SJ_A4.2, U1.A4
- removed net A5: R13.2, SJ_A5.2, U1.A5
- removed net VCC: C20.P$1, R20.2, R21.2, SJ_A0.1, SJ_A1.1, SJ_A2.1, SJ_A3.1, SJ_A4.1, SJ_A5.1, U1.VDD
- new net IR_IN: IR-RECEIVER-3.S, JP7.3
- new net PWM5: U1.PWM5
- net 0_PWM: now also R11.1; no longer R5.1
- net 1_PWM: now also R9.1; no longer R7.1
- net 2_PWM: now also R7.1; no longer R9.1
- net 3V3: now also 0604.2, C20.P$1, C3.2, C6.+, D1.A, IC1.FB, IR-RECEIVER-1.S, JP2.1, MOTOR-1.S, R20.2, R21.2, U$4.A, U1.A0, U1.A2, U1.A4, U1.VDD; no longer JP1.1, JP5.22
- net 3_PWM: now also R5.1; no longer R11.1
- net GND: now also IR-RECEIVER-2.S, U1.A1, U1.A3, U1.A5; no longer R13.1, R14.1, R15.1, R16.1, R17.1, R18.1
- net M-: now also MOTOR-2.S; no longer JP1.2, X3.2
- net M_PWM: now also U1.PWM4; no longer U1.PWM5, X3.1
Other:
- note removed: "1 + A5 + A4 + A3 + A2 + A1 +A1 + RW"
- note removed: "Check sda scl polarity"
- note removed: "I2C Address ="
- note removed: "M+"
- note removed: "Open = 0 / Closed = 1"

Commit message: changes added polygon and some changes for version1
Connections:
- net +24V_EINGANG renamed VIN24V
Other:
- note removed: "!! Check Footprints they are random."
- moved on the sheet: C20, R19, R20, R21, U1
